File: KiCad/ReAgnus-MegAChip_FPGA.sch (KiCad schematic (older format))
At the start: 18 parts, among them J2 Conn_02x05_Odd_Even, J3 Conn_02x02_Odd_Even, U1 GW1NR-UV9LQ144P, U10 74LVC245A, U11 MCP1702T-1802E_CB, U9 74LVC1GX04, Y1 CL=16pF

Commit message: Changed L1 from inductor to ferrite bead 600 Ohms impedance, changed C6 to 10uF, C9 to 1uF, C27 to 0.1uF, C28 to 0.1uF
Parts:
- C28: value 0.01uF -> 0.1uF
- C6: value 0.1uF -> 10uF
- L1: value 10uH -> 600
Changed lines of the file:
@@
 AR Path="/632F104D/66807BC8" Ref="C6"  Part="1"
 F 0 "C6" H 8550 5200 50  0000 L CNN
-F 1 "0.1uF" H 8600 5100 50  0001 L CNN
+F 1 "10uF" H 8600 5100 50  0001 L CNN
 F 2 "Capacitor_SMD:C_0805_2012Metric_Pad1.18x1.45mm_HandSolder" H 8600 5350 50  0001 C CNN
 F 3 "~" H 8600 5350 50  0001 C CNN
@@
 P 8350 5450
 F 0 "L1" V 8300 5400 50  0000 L CNN
-F 1 "10uH" V 8450 5350 50  0000 L CNN
+F 1 "600" V 8450 5400 50  0000 L CNN
 F 2 "Inductor_SMD:L_0805_2012Metric_Pad1.05x1.20mm_HandSolder" H 8350 5450 50  0001 C CNN
 F 3 "~" H 8350 5450 50  0001 C CNN
@@
 AR Path="/632F104D/668717A8" Ref="C28"  Part="1"
 F 0 "C28" H 7850 5400 50  0000 L CNN
-F 1 "0.01uF" H 8100 5100 50  0001 L CNN
+F 1 "0.1uF" H 8100 5100 50  0001 L CNN
 F 2 "Capacitor_SMD:C_0603_1608Metric_Pad1.08x0.95mm_HandSolder" H 8100 5350 50  0001 C CNN
 F 3 "~" H 8100 5350 50  0001 C CNN
@@
 Wire Wire Line
 	8100 5250 8600 5250
-Text GLabel 7950 5450 0    50   Output ~ 0
-VCCIO3
 Text GLabel 10200 1450 3    50   Input ~ 0
 TDO
@@
 	-1   0    0    1
 $EndComp
+Text GLabel 7950 5450 0    50   Output ~ 0
+VCCIO3
 $EndSCHEMATC
